File: SI-P Pressure Transducer/SI-P Pressure Transducer.kicad_pcb (KiCad board)
At the start: 2 copper layers, 32.6 x 17.8 mm, 24 parts, among them J1 Conn_01x06_Pin, J2 Conn_01x06_Socket, J3 Screw_Terminal_01x02, J4 AVR-ISP-6, U1 ATtiny841-SS, U2 LM2621MM/NOPB

Commit message: First revision of boards
Parts:
- removed J3: Screw_Terminal_01x02, TerminalBlock:TerminalBlock_bornier-2_P5.08mm
- added J5: Screw_Terminal_01x03, TerminalBlock_Phoenix:TerminalBlock_Phoenix_MPT-0,5-3-2.54_1x03_P2.54mm_Horizontal, F.Cu at (185.4, 73.5)
- added R10: 1k, Resistor_SMD:R_0603_1608Metric, F.Cu at (193.5, 71.7)
- added R9: 3.9k, Resistor_SMD:R_0603_1608Metric, F.Cu at (191.0, 69.0)
- C3: footprint Capacitor_SMD:C_0603_1608Metric -> Capacitor_SMD:C_0805_2012Metric
- moved C5 0.70 mm to (200.5, 64.0)
- moved C3 0.27 mm to (198.5, 63.8)
- moved R4 0.10 mm to (200.6, 61.4)
Connections:
- U1 pad 3: unconnected-(U1-XTAL2/PB1-Pad3) -> Net-(U1-XTAL2/PB1)
Routing:
- net Net-(U1-XTAL2/PB1): track 0.00 -> 17.0 mm, vias 0 -> 2
- net GND: track 105.3 -> 112.0 mm
- net +12V: track 47.5 -> 53.9 mm
- net +3V3: track 78.8 -> 81.3 mm
- net /PT_OUT: track 24.2 -> 26.0 mm
- net /I2C_SDA: track 38.8 -> 37.1 mm
- net Net-(U2-VDD): track 10.1 -> 11.4 mm
- net /STATUS: track 56.4 -> 57.4 mm
Other:
- board size 32.6 x 17.8 mm -> 33.1 x 17.8 mm
