File: SI-P Pressure Transducer/SI-P Pressure Transducer.kicad_sch (KiCad schematic)
At the start: 24 parts, among them J1 Conn_01x06_Pin, J2 Conn_01x06_Socket, J3 Screw_Terminal_01x02, J4 AVR-ISP-6, U1 ATtiny841-SS, U2 LM2621MM/NOPB

Commit message: First revision of boards
Parts:
- removed J3: Screw_Terminal_01x02, TerminalBlock:TerminalBlock_bornier-2_P5.08mm, symbol Connector:Screw_Terminal_01x02
- added J5: Screw_Terminal_01x03, TerminalBlock_Phoenix:TerminalBlock_Phoenix_MPT-0,5-3-2.54_1x03_P2.54mm_Horizontal, symbol Connector:Screw_Terminal_01x03
- added R10: 1k, Resistor_SMD:R_0603_1608Metric, symbol Device:R
- added R9: 3.9k, Resistor_SMD:R_0603_1608Metric, symbol Device:R
- C3: footprint Capacitor_SMD:C_0603_1608Metric -> Capacitor_SMD:C_0805_2012Metric
Connections:
- net +12V: now also J5.2 (Pin_2), J5.3 (Pin_3), R9.1
- net GND: now also R10.2
- net PT_OUT: now also J5.1 (Pin_1)
- net at U1.3 (XTAL2/PB1): now also R10.1, R9.2
- no-connect marks 2 -> 1
